Commit message: added new controllers

File: resources/robots/x500arm/model.urdf (robot description, URDF)
Before this commit: robot quadrotor_with_arm, 8 links, 7 joints
Links:
- removed link arm_base_link
- removed link arm_link_1
- removed link arm_link_2
- added link l1_link, mass 0.052; collision cylinder length=0.038 radius=0.02; visual cylinder length=0.038 radius=0.02
- added link l2_link, mass 0.038; collision cylinder length=0.236 radius=0.02; visual cylinder length=0.236 radius=0.02
- added link l3_link, mass 0.219; collision cylinder length=0.216 radius=0.02; visual cylinder length=0.216 radius=0.02
- added link l4_link, mass 0.05; collision box size=0.02 0.06 0.04; visual box size=0.02 0.06 0.04
- link back_left_prop: mass 0.064 -> 0.016076923076923075; geometry visual cylinder length=0.01 radius=0.13
- link back_right_prop: mass 0.064 -> 0.016076923076923075; geometry visual cylinder length=0.01 radius=0.13
- link base_link: mass 1.4 -> 2.0; geometry collision box size=0.353 0.353 0.05; visual box size=0.353 0.353 0.05
- link front_left_prop: mass 0.064 -> 0.016076923076923075; geometry visual cylinder length=0.01 radius=0.13
- link front_right_prop: mass 0.064 -> 0.016076923076923075; geometry visual cylinder length=0.01 radius=0.13
Joints:
- removed joint joint_1
- removed joint joint_2
- removed joint mount_joint
- added joint L1_to_L2: type revolute, parent l1_link, child l2_link, origin xyz=0 0 0.03796 rpy=0 1.57 0, axis 0 1 0, limit lower=-3.14 upper=0 effort=1000 velocity=0.5
- added joint L2_to_L3: type revolute, parent l2_link, child l3_link, origin xyz=0.03 0 0.23682 rpy=0 0 0, axis 0 1 0, limit lower=-3.14 upper=3.14 effort=1000 velocity=0.5
- added joint L3_to_L4: type revolute, parent l3_link, child l4_link, origin xyz=0 0 0.21599 rpy=0 0 0, axis 0 0 1, limit lower=-3.14 upper=3.14 effort=1000 velocity=0.5
- added joint arm_to_L1: type fixed, parent base_link, child l1_link, origin xyz=0 0 -0.025 rpy=0 3.14159265 0
- joint base_link_to_back_left_prop: origin xyz=-0.174 0.174 0 -> xyz=-0.174 0.174 0.06
- joint base_link_to_back_right_prop: origin xyz=-0.174 -0.174 0 -> xyz=-0.174 -0.174 0.06
- joint base_link_to_front_left_prop: origin xyz=0.174 0.174 0 -> xyz=0.174 0.174 0.06
- joint base_link_to_front_right_prop: origin xyz=0.174 -0.174 0 -> xyz=0.174 -0.174 0.06
