Commit message: added il_control

File: resources/robots/x500/model.urdf (robot description, URDF)
Before this commit: robot quadrotor, 5 links, 4 joints
Links:
- link base_link: mass 1.4 -> 1.772
Joints:
- joint base_link_to_back_left_prop: origin xyz=-0.174 0.174 0 -> xyz=-0.22 0.22 0
- joint base_link_to_back_right_prop: origin xyz=-0.174 -0.174 0 -> xyz=-0.22 -0.22 0
- joint base_link_to_front_left_prop: origin xyz=0.174 0.174 0 -> xyz=0.22 0.22 0
- joint base_link_to_front_right_prop: origin xyz=0.174 -0.174 0 -> xyz=0.22 -0.22 0

File: resources/robots/x500arm/model.urdf (robot description, URDF)
Before this commit: robot quadrotor_with_arm, 9 links, 8 joints
Links:
- link base_link: geometry collision box size=1.0 1.0 0.05; visual box size=0.353 0.353 0.05
